Commit message: Add new meshes and update kinematic scheme

File: urdf/tinybot.urdf.xacro (robot description, xacro)
@@ -6,9 +6,9 @@
 -->
   <xacro:macro name="tinybot_urdf" params="prefix
-    joint1_lower_limit:=${-2.0*pi}  joint1_upper_limit:=${2.0*pi}
-    joint2_lower_limit:=${-2.059}  joint2_upper_limit:=${2.0944}
-    joint3_lower_limit:=${-3.927}  joint3_upper_limit:=${0.19198}
-    joint4_lower_limit:=${-1.69297}  joint4_upper_limit:=${pi}
-    joint5_lower_limit:=${-2.0*pi}  joint5_upper_limit:=${2.0*pi}">
+    joint1_lower_limit:=${-pi}  joint1_upper_limit:=${pi}
+    joint2_lower_limit:=${-pi}  joint2_upper_limit:=${pi}
+    joint3_lower_limit:=${-pi}  joint3_upper_limit:=${pi}
+    joint4_lower_limit:=${-pi}  joint4_upper_limit:=${pi}
+    joint5_lower_limit:=${-pi}  joint5_upper_limit:=${pi}">
     <material name="Black">
       <color rgba="0.0 0.0 0.0 1.0"/>
@@ -24,221 +24,325 @@
     </material>
     <!-- Base link -->
-    <link name="${prefix}base_link">
-      <inertial>
-        <origin
-          xyz="-0.00218 -0.00023 0.08604" rpy="0 0 0" />
-        <mass value="1.95" />
-        <inertia
-          ixx="0.004805" ixy="-8.33E-06" ixz="0.00026847"
-          iyy="0.0050349" iyz="7.23E-06" izz="0.0025418"/>
-      </inertial>
-      <visual>
-        <origin xyz="0 0 0" rpy="0 0 0" />
-        <geometry>
-          <mesh filename="package://tinybot_description/meshes/base_link.STL" scale="0.001 0.001 0.001"/>
-        </geometry>
-        <material name="White" />
-      </visual>
-      <collision>
-        <origin xyz="0 0 0" rpy="0 0 0" />
-        <geometry>
-          <mesh filename="package://tinybot_description/meshes/base_link.STL" scale="0.001 0.001 0.001"/>
-        </geometry>
-      </collision>
-    </link>
-    <!-- Link 1 -->
-    <link name="${prefix}link1">
-      <inertial>
-        <origin xyz="0.00016 0.02064 -0.01556" rpy="0 0 0" />
-        <mass value="1.85" />
-        <inertia
-          ixx="0.0046885" ixy="-8.67E-06" ixz="2.439E-05"
-          iyy="0.0041688" iyz="0.0006114" izz="0.0024758" />
-      </inertial>
-      <visual>
-        <origin xyz="0 0 0" rpy="0 0 0" />
-        <geometry>
-          <mesh filename="package://tinybot_description/meshes/link1.STL" scale="0.001 0.001 0.001"/>
-        </geometry>
-        <material name="White" />
-      </visual>
-      <collision>
-        <origin xyz="0 0 0" rpy="0 0 0" />
-        <geometry>
-          <mesh filename="package://tinybot_description/meshes/link1.STL" scale="0.001 0.001 0.001"/>
-        </geometry>
-      </collision>
-    </link>
-    <!-- Joint 1 -->
-    <joint name="${prefix}joint1" type="revolute">
-      <origin xyz="0 0 0.101" rpy="0 0 0" />
-      <parent link="${prefix}base_link" />
-      <child link="${prefix}link1" />
-      <axis xyz="0 0 1" />
-     <limit
+    <link
+    name="${prefix}base_link">
+    <inertial>
+      <origin
+        xyz="1.8574E-07 9.9166E-05 0.040638"
+        rpy="0 0 0" />
+      <mass
+        value="1.999" />
+      <inertia
+        ixx="0.00069146"
+        ixy="8.8315E-09"
+        ixz="-4.3606E-10"
+        iyy="0.00070155"
+        iyz="4.9309E-07"
+        izz="0.0012677" />
+    </inertial>
+    <visual>
+      <origin
+        xyz="0 0 0"
+        rpy="0 0 0" />
+      <geometry>
+        <mesh
+          filename="package://tinybot_description/meshes/base_link.STL" />
+      </geometry>
+      <material
+        name="">
+        <color
+          rgba="0.6902 0.6902 0.6902 1" />
+      </material>
+    </visual>
+    <collision>
+      <origin
+        xyz="0 0 0"
+        rpy="0 0 0" />
+      <geometry>
+        <mesh
+          filename="package://tinybot_description/meshes/base_link.STL" />
+      </geometry>
+    </collision>
+  </link>
+  <link
+    name="${prefix}link1">
+    <inertial>
+      <origin
+        xyz="0.00053822 -0.0030286 0.057419"
+        rpy="0 0 0" />
+      <mass
+        value="1.962" />
+      <inertia
+        ixx="0.00020802"
+        ixy="5.8641E-07"
+        ixz="-8.8309E-09"
+        iyy="0.00033929"
+        iyz="-4.3611E-10"
+        izz="0.00021938" />
+    </inertial>
+    <visual>
+      <origin
+        xyz="0 0 0"
+        rpy="0 0 0" />
+      <geometry>
+        <mesh
+          filename="package://tinybot_description/meshes/link1.STL" />
+      </geometry>
+      <material
+        name="">
+        <color
+          rgba="0.52941 0.54902 0.54902 1" />
+      </material>
+    </visual>
+    <collision>
+      <origin
+        xyz="0 0 0"
+        rpy="0 0 0" />
+      <geometry>
+        <mesh
+          filename="package://tinybot_description/meshes/link1.STL" />
+      </geometry>
+    </collision>
+  </link>
+  <joint
+    name="joint1"
+    type="revolute">
+    <origin
+      xyz="0 0 0.1015"
+      rpy="0 0 0" />
+    <parent
+      link="base_link" />
+    <child
+      link="link1" />
+    <axis
+      xyz="0 0 1" />
+    <limit
         lower="${joint1_lower_limit}"
         upper="${joint1_upper_limit}"
         effort="50"
-        velocity="3.14" />
-      <dynamics
-        damping="10"
-        friction="1" />
-    </joint>
-    <!-- Link 2 -->
-    <link name="${prefix}link2">
-      <inertial>
-        <origin xyz="0.0351 -0.21375 0.02835" rpy="0 0 0" />
-        <mass value="1.71" />
-        <inertia
-          ixx="0.024904" ixy="-0.004271" ixz="-0.0008356"
-          iyy="0.004901" iyz="0.0052393" izz="0.0238188" />
-      </inertial>
-      <visual>
-        <origin xyz="0 0 0" rpy="0 0 0" />
-        <geometry>
-          <mesh filename="package://tinybot_description/meshes/link2.STL" scale="0.001 0.001 0.001"/>
-        </geometry>
-        <material name="White" />
-      </visual>
-      <collision>
-        <origin xyz="0 0 0" rpy="0 0 0" />
-        <geometry>
-          <mesh filename="package://tinybot_description/meshes/link2.STL" scale="0.001 0.001 0.001"/>
-        </geometry>
-      </collision>
-    </link>
-    <!-- Joint 2 -->
-    <joint name="${prefix}joint2" type="revolute">
-      <origin xyz="0.0325 0 0.0665" rpy="0 -1.5708 0" />
-      <parent link="${prefix}link1" />
-      <child link="${prefix}link2" />
-      <axis xyz="0 0 1" />
-      <limit
+        velocity="1.0" />
+      <dynamics
+        damping="5"
+        friction="1" />
+  </joint>
+  <link
+    name="link2">
+    <inertial>
+      <origin
+        xyz="0.12597 8.5763E-10 0.024345"
+        rpy="0 0 0" />
+      <mass
+        value="0.778" />
+      <inertia
+        ixx="0.00012535"
+        ixy="1.2464E-11"
+        ixz="1.3405E-10"
+        iyy="0.0013458"
+        iyz="1.6238E-10"
+        izz="0.001368" />
+    </inertial>
+    <visual>
+      <origin
+        xyz="0 0 0"
+        rpy="0 0 0" />
+      <geometry>
+        <mesh
+          filename="package://tinybot_description/meshes/link2.STL" />
+      </geometry>
+      <material
+        name="">
+        <color
+          rgba="1 1 1 1" />
+      </material>
+    </visual>
+    <collision>
+      <origin
+        xyz="0 0 0"
+        rpy="0 0 0" />
+      <geometry>
+        <mesh
+          filename="package://tinybot_description/meshes/link2.STL" />
+      </geometry>
+    </collision>
+  </link>
+  <joint
+    name="${prefix}joint2"
+    type="revolute">
+    <origin
+      xyz="0 -0.032 0.068"
+      rpy="1.5708 -1.5708 0" />
+    <parent
+      link="${prefix}link1" />
+    <child
+      link="${prefix}link2" />
+    <axis
+      xyz="0 0 1" />
+    <limit
         lower="${joint2_lower_limit}"
         upper="${joint2_upper_limit}"
         effort="50"
-        velocity="3.14" />
-      <dynamics
-        damping="10"
-        friction="1" />
-    </joint>
-    <!-- Link 3 -->
-    <link name="${prefix}link3">
-      <inertial>
-        <origin xyz="0.06716 0.2299 -0.00249" rpy="0 0 0" />
-        <mass value="1.74" />
-        <inertia
-          ixx="0.0335922" ixy="0.0040788" ixz="-0.0014658"
-          iyy="0.0055857" iyz="-0.0080609" izz="0.0318905" />
-      </inertial>
-      <visual>
-        <origin
-          xyz="0 0 0"
-          rpy="0 0 0" />
-        <geometry>
-          <mesh
-            filename="package://tinybot_description/meshes/link3.STL" scale="0.001 0.001 0.001"/>
-        </geometry>
-        <material name="White" />
-      </visual>
-      <collision>
-        <origin
-          xyz="0 0 0"
-          rpy="0 0 0" />
-        <geometry>
-          <mesh
-            filename="package://tinybot_description/meshes/link3.STL" scale="0.001 0.001 0.001"/>
-        </geometry>
-      </collision>
-    </link>
-    <joint
-      name="${prefix}joint3"
-      type="revolute">
-      <origin
-        xyz="0.0 0.250 0.0"
-        rpy="0 0 0" />
-      <parent
-        link="${prefix}link2" />
-      <child
-        link="${prefix}link3" />
-      <axis
-        xyz="0 0 1" />
-      <limit
+        velocity="1.0" />
+      <dynamics
+        damping="5"
+        friction="1" />
+  </joint>
+  <link
+    name="${prefix}link3">
+    <inertial>
+      <origin
+        xyz="0.16701 -0.00035709 -0.024615"
+        rpy="0 0 0" />
+      <mass
+        value="2.849" />
+      <inertia
+        ixx="0.00033763"
+        ixy="-1.9393E-10"
+        ixz="1.2229E-09"
+        iyy="0.00073725"
+        iyz="2.8549E-06"
+        izz="0.00082439" />
+    </inertial>
+    <visual>
+      <origin
+        xyz="0 0 0"
+        rpy="0 0 0" />
+      <geometry>
+        <mesh
+          filename="package://tinybot_description/meshes/link3.STL" />
+      </geometry>
+      <material
+        name="">
+        <color
+          rgba="0.8 0.8 0.8 1" />
+      </material>
+    </visual>
+    <collision>
+      <origin
+        xyz="0 0 0"
+        rpy="0 0 0" />
+      <geometry>
+        <mesh
+          filename="package://tinybot_description/meshes/link3.STL" />
+      </geometry>
+    </collision>
+  </link>
+  <joint
+    name="${prefix}joint3"
+    type="revolute">
+    <origin
+      xyz="0.24998 0 0"
+      rpy="0 0 0" />
+    <parent
+      link="${prefix}link2" />
+    <child
+      link="${prefix}link3" />
+    <axis
+      xyz="0 0 1" />
+    <limit
         lower="${joint3_lower_limit}"
         upper="${joint3_upper_limit}"
-        effort="30"
-        velocity="3.14" />
-      <dynamics
-        damping="5"
-        friction="1" />
-    </joint>
-    <link
-      name="${prefix}link4">
-      <inertial>
-        <origin
-          xyz="0.0636 0.02203 0.00355"
-          rpy="0 0 0" />
-        <mass
-          value="1.13" />
-        <inertia
-          ixx="0.0010927"
-          ixy="0.0003076"
-          ixz="-0.0002076"
-          iyy="0.0016058"
-          iyz="-8.863E-05"
-          izz="0.0019148" />
-      </inertial>
-      <visual>
-        <origin
-          xyz="0 0 0"
-          rpy="0 0 0" />
-        <geometry>
-          <mesh
-            filename="package://tinybot_description/meshes/link4.STL" scale="0.001 0.001 0.001"/>
-        </geometry>
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
File: urdf/tinybot_macro.xacro (robot description, xacro)
@@ -23,9 +23,9 @@
     <xacro:if value="${limited}">
       <xacro:tinybot_urdf prefix="${prefix}"
-        joint1_lower_limit="${-pi*0.99}" joint1_upper_limit="${pi*0.99}"
-        joint2_lower_limit="${-2.059}" joint2_upper_limit="${2.0944}"
-        joint3_lower_limit="${-pi*0.99}" joint3_upper_limit="${0.19198}"
-        joint4_lower_limit="${-1.69297}" joint4_upper_limit="${pi*0.99}"
-        joint5_lower_limit="${-pi*0.99}" joint5_upper_limit="${pi*0.99}"/>
+        joint1_lower_limit="${-pi}" joint1_upper_limit="${pi}"
+        joint2_lower_limit="${-0.5*pi}" joint2_upper_limit="${0.5*pi}"
+        joint3_lower_limit="${-0.75*pi}" joint3_upper_limit="${0.75*pi}"
+        joint4_lower_limit="${-0.75*pi}" joint4_upper_limit="${0.75*pi}"
+        joint5_lower_limit="${-pi}" joint5_upper_limit="${pi}"/>
     </xacro:if>
     <xacro:unless value="${limited}">
